Commit message: hand_motor_joint, hand_l_spring_proximal_joint, hand_r_spring_proximal_joint: fixed -> revolute

File: hsrb_description/robots/hsrb4s.urdf (robot description, URDF)
Before this commit: robot hsrb, 51 links, 50 joints
Joints:
- joint hand_l_spring_proximal_joint: type fixed -> revolute
- joint hand_motor_joint: type fixed -> revolute
- joint hand_r_spring_proximal_joint: type fixed -> revolute

Commit message: made some stuff similar to original urdf, cut out extra tags
urdf used as reference is https://github.com/hsr-project/hsrb_description/blob/master/robots/hsrb4s.urdf

File: hsrb_description/robots/hsrb4s.urdf (robot description, URDF)
Before this commit: robot hsrb, 51 links, 50 joints
Links:
- link hand_l_distal_link: geometry collision mesh filename=package://hsrb_meshes/meshes/hand_v0/l_distal.stl; visual mesh filename=package://hsrb_meshes/meshes/hand_v0/l_distal.dae
- link hand_l_spring_proximal_link: geometry collision mesh filename=package://hsrb_meshes/meshes/hand_v0/l_proximal.stl; visual mesh filename=package://hsrb_meshes/meshes/hand_v0/l_proximal.dae
- link hand_r_distal_link: geometry collision mesh filename=package://hsrb_meshes/meshes/hand_v0/r_distal.stl; visual mesh filename=package://hsrb_meshes/meshes/hand_v0/r_distal.dae
- link hand_r_spring_proximal_link: geometry collision mesh filename=package://hsrb_meshes/meshes/hand_v0/r_proximal.stl; visual mesh filename=package://hsrb_meshes/meshes/hand_v0/r_proximal.dae
Joints:
- joint hand_l_distal_joint: limit lower=-1.24 upper=0.798 effort=100.0 velocity=5.0 -> lower=-1.24 upper=0.798 effort=100.0 velocity=1.0
- joint hand_l_mimic_distal_joint: type fixed -> revolute
- joint hand_l_proximal_joint: limit lower=-0.798 upper=1.24 effort=1.0 velocity=5.0 -> lower=-0.798 upper=1.24 effort=100.0 velocity=1.0
- joint hand_l_spring_proximal_joint: limit lower=0.0 upper=0.698 effort=1.0 velocity=1.0 -> lower=0.0 upper=0.698 effort=10.0 velocity=1.0
- joint hand_r_distal_joint: limit lower=-1.24 upper=0.798 effort=100.0 velocity=5.0 -> lower=-1.24 upper=0.798 effort=100.0 velocity=1.0
- joint hand_r_mimic_distal_joint: limit lower=-0.698 upper=-0.0 effort=100.0 velocity=5.0 -> lower=-0.698 upper=-0.0 effort=100.0 velocity=1.0; type fixed -> revolute
- joint hand_r_proximal_joint: limit lower=-0.798 upper=1.24 effort=1.0 velocity=5.0 -> lower=-0.798 upper=1.24 effort=100.0 velocity=1.0
- joint hand_r_spring_proximal_joint: limit lower=0.0 upper=0.698 effort=1.0 velocity=1.0 -> lower=0.0 upper=0.698 effort=10.0 velocity=1.0
- joint torso_lift_joint: limit lower=0.0 upper=0.345 effort=1000.0 velocity=0.1 -> lower=0.0 upper=0.345 effort=300.0 velocity=0.1

Commit message: increases efforts, reduces ROM, changes revolute -> fixed

File: hsrb_description/robots/hsrb4s.urdf (robot description, URDF)
Before this commit: robot hsrb, 51 links, 50 joints
Joints:
- joint hand_l_distal_joint: type revolute -> fixed
- joint hand_l_mimic_distal_joint: type revolute -> fixed
- joint hand_l_proximal_joint: limit lower=-0.798 upper=1.24 effort=100.0 velocity=1.0 -> lower=0 upper=0.7 effort=100.0 velocity=1.0
- joint hand_l_spring_proximal_joint: limit lower=0.0 upper=0.698 effort=10.0 velocity=1.0 -> lower=0.0 upper=0.698 effort=1.0 velocity=1.0; type revolute -> fixed
- joint hand_motor_joint: limit lower=-0.798 upper=1.24 effort=100.0 velocity=1.0 -> lower=0 upper=1.24 effort=1000.0 velocity=1.0; type revolute -> fixed
- joint hand_r_distal_joint: type revolute -> fixed
- joint hand_r_mimic_distal_joint: limit lower=-0.698 upper=-0.0 effort=100.0 velocity=1.0 -> lower=-0.698 upper=-0.0 effort=100.0 velocity=5.0; type revolute -> fixed
- joint hand_r_proximal_joint: limit lower=-0.798 upper=1.24 effort=100.0 velocity=1.0 -> lower=0 upper=0.7 effort=100.0 velocity=1.0
- joint hand_r_spring_proximal_joint: limit lower=0.0 upper=0.698 effort=10.0 velocity=1.0 -> lower=0.0 upper=0.698 effort=1.0 velocity=1.0; type revolute -> fixed
